Commit message: custom joint and link

File: models/robot.xacro (robot description, xacro)
@@ -2,37 +2,136 @@
 <robot name="spw_robot" xmlns:xacro="http://www.ros.org/wiki/xacro">
   <xacro:include filename="$(find spw_robot)/models/robot.gazebo" />
-  <gazebo reference="left_wheel">
-    <material>Gazebo/Green</material>
-  </gazebo>
-  <gazebo reference="right_wheel">
-    <material>Gazebo/Green</material>
-  </gazebo>
-  <gazebo reference="camera">
-    <material>Gazebo/Red</material>
-  </gazebo>
-  <gazebo reference="chassis">
-    <material>Gazebo/Blue</material>
-  </gazebo>
+  <gazebo reference="base_center"><material>Gazebo/Blue</material></gazebo>
+  <gazebo reference="left_wheel"><material>Gazebo/Black</material></gazebo>
+  <gazebo reference="right_wheel"><material>Gazebo/Black</material></gazebo>
+  <gazebo reference="link1"><material>Gazebo/Grey</material></gazebo>
+  <gazebo reference="link2"><material>Gazebo/Grey</material></gazebo>
+  <gazebo reference="link3"><material>Gazebo/Grey</material></gazebo>
+  <!-- FOOT PRINT -->
   <link name="robot_footprint"></link>
   <joint name="robot_footprint_joint" type="fixed">
     <origin xyz="0 0 0" rpy="0 0 0" />
     <parent link="robot_footprint"/>
-    <child link="chassis" />
+    <child link="base_center" />
   </joint>
-  <joint name="camera_joint" type="fixed">
-    <origin xyz="0.26 0 0" rpy="0 0 0" />
-    <parent link="chassis"/>
-    <child link="camera" />
+  <!-- BASE -->
+  <link name="base_center">
+    <pose>0 0 0.1 0 0 0</pose>
+    <inertial>
+      <mass value="15.0"/>
+      <origin xyz="0.0 0 0" rpy=" 0 0 0"/>
+      <inertia
+          ixx="0.1" ixy="0" ixz="0"
+          iyy="0.1" iyz="0"
+          izz="0.1"
+      />
+    </inertial>
+    <collision name="collision">
+      <origin xyz="0 0 0.05" rpy=" 0 0 0"/>
+      <geometry>
+        <box size="1 1 1"/>
+      </geometry>
+    </collision>
+    <visual name="base_center_visual">
+      <origin xyz="0 0 0.05" rpy=" 0 0 0"/>
+      <geometry>
+        <box size="1 1 1"/>
+      </geometry>
+    </visual>
+  </link>
+  <!-- ARM TO ROTATE Z AXIS -->
+  <joint name="joint1" type="revolute">
+    <parent link="base_center"/>
+    <child link="link1"/>
+    <origin xyz="0 0 1" rpy="0 0 0"/>
+    <axis xyz="0 0 1"/>
+    <limit effort="100" velocity="100" lower="-1.5708" upper="1.5708"/>
+  </joint>
+  <link name="link1">
+    <collision>
+      <origin xyz="0 0 0.05" rpy="0 0 0"/>
+      <geometry>
+        <cylinder length="1" radius="0.2"/>
+      </geometry>
+    </collision>
+    <visual>
+      <origin xyz="0 0 0.05" rpy="0 0 0"/>
+      <geometry>
+        <cylinder length="1" radius="0.2"/>
+      </geometry>
+    </visual>
+    <inertial>
+      <origin xyz="0 0 0.05" rpy="0 0 0"/>
+      <mass value="1"/>
+      <inertia
+        ixx="0.001" ixy="0.0" ixz="0.0"
+        iyy="0.001" iyz="0.0"
+        izz="0.001"/>
+    </inertial>
+  </link>
+  <!-- ARM TO ROTATE Y AXIS -->
+  <joint name="joint2" type="revolute">
+    <parent link="link1"/>
+    <child link="link2"/>
+    <origin xyz="0 0 0.1" rpy="0 0 0"/>
     <axis xyz="0 1 0"/>
+    <limit effort="100" velocity="100" lower="-0.1" upper="1.5708"/>
   </joint>
-  <joint name="hokuyo_joint" type="fixed">
-    <origin xyz="0.2 0 0.2" rpy="0 0 0" />
-    <parent link="chassis"/>
-    <child link="hokuyo" />
+  <link name="link2">
+    <collision>
+      <origin xyz="0 0 0.5" rpy="0 0 0"/>
+      <geometry>
+        <cylinder length="1" radius="0.1"/>
+      </geometry>
+    </collision>
+    <visual>
+      <origin xyz="0 0 0.5" rpy="0 0 0"/>
+      <geometry>
+        <cylinder length="1" radius="0.1"/>
+      </geometry>
+    </visual>
+    <inertial>
+      <origin xyz="0 0 0.5" rpy="0 0 0"/>
+      <mass value="1"/>
+      <inertia
+        ixx="0.1" ixy="0.0" ixz="0.0"
+        iyy="0.1" iyz="0.0"
+        izz="0.005"/>
+    </inertial>
+  </link>
+  <!-- ARM TO ROTATE X AXIS -->
+  <joint name="joint3" type="revolute">
+    <parent link="link2"/>
+    <child link="link3"/>
+    <origin xyz="0 0 1" rpy="0 0 0"/>
     <axis xyz="0 1 0"/>
+    <limit effort="100" velocity="100" lower="-0.1" upper="3.1416"/>
   </joint>
-  <joint type="continuous" name="left_wheel_hinge">
-    <origin xyz="0 0.30 0" rpy="0 0 0" />
-    <parent link="chassis"/>
+  <link name="link3">
+    <collision>
+      <origin xyz="0 0 0.5" rpy="0 0 0"/>
+      <geometry>
+        <cylinder length="1" radius="0.1"/>
+      </geometry>
+    </collision>
+    <visual>
+      <origin xyz="0 0 0.5" rpy="0 0 0"/>
+      <geometry>
+        <cylinder length="1" radius="0.1"/>
+      </geometry>
+    </visual>
+    <inertial>
+      <origin xyz="0 0 0.5" rpy="0 0 0"/>
+      <mass value="1"/>
+      <inertia
+        ixx="0.1" ixy="0.0" ixz="0.0"
+        iyy="0.1" iyz="0.0"
+        izz="0.005"/>
+    </inertial>
+  </link>
+  <!-- WHEELS -->
+  <joint name="left_wheel_hinge" type="continuous">
+    <origin xyz="0 0.5 0" rpy="0 0 0" />
+    <parent link="base_center"/>
     <child link="left_wheel" />
     <axis xyz="0 1 0" rpy="0 0 0" />
@@ -40,7 +139,7 @@
     <dynamics damping="1.0" friction="1.0" />
   </joint>
-  <joint type="continuous" name="right_wheel_hinge">
-    <origin xyz="0 -0.30 0" rpy="0 0 0" />
-    <parent link="chassis"/>
+  <joint name="right_wheel_hinge" type="continuous">
+    <origin xyz="0 -0.5 0" rpy="0 0 0" />
+    <parent link="base_center"/>
     <child link="right_wheel" />
     <axis xyz="0 1 0" rpy="0 0 0" />
@@ -48,50 +147,4 @@
     <dynamics damping="1.0" friction="1.0" />
   </joint>
-<link name="camera">
-    <inertial>
-      <mass value="0.1"/>
-      <origin xyz="0 0 0" rpy="0 0 0"/>
-      <inertia
-        ixx="1e-6" ixy="0.0" ixz="0.0"
-        iyy="1e-6" iyz="0.0"
-        izz="1e-6"
-      />
-    </inertial>
-    <collision>
-      <origin xyz="0 0 0" rpy="0 0 0"/>
-      <geometry>
-        <box size="0.05 0.05 0.05"/>
-      </geometry>
-    </collision>
-    <visual>
-      <origin xyz="0 0 0" rpy="0 0 0"/>
-      <geometry>
-        <box size="0.05 0.05 0.05"/>
-      </geometry>
-    </visual>
-  </link>
-  <link name="hokuyo">
-    <inertial>
-      <mass value="1e-5"/>
-      <origin xyz="0 0 0" rpy="0 0 0"/>
-      <inertia
-        ixx="1e-6" ixy="0.0" ixz="0.0"
-        iyy="1e-6" iyz="0.0"
-        izz="1e-6"
-      />
-    </inertial>
-    <collision>
-      <origin xyz="0 0 0" rpy="0 0 0"/>
-      <geometry>
-        <box size="0.1 0.1 0.1"/>
-      </geometry>
-    </collision>
-    <!-- <visual>
-      <origin xyz="0 0 0" rpy="0 0 0"/>
-      <geometry>
-        <mesh filename="package://trixy/meshes/hokuyo.dae"/>
-      </geometry>
-    </visual> -->
-  </link>
   <link name="left_wheel">
     <inertial>
@@ -107,5 +160,5 @@
       <origin xyz="0 0 0" rpy="0 1.5707 1.5707"/>
       <geometry>
-        <cylinder radius="0.1" length="0.05"/>
+        <cylinder radius="0.5" length="0.5"/>
       </geometry>
     </collision>
@@ -113,5 +166,5 @@
       <origin xyz="0 0 0" rpy="0 1.5707 1.5707"/>
       <geometry>
-        <cylinder radius="0.1" length="0.05"/>
+        <cylinder radius="0.5" length="0.5"/>
       </geometry>
     </visual>
@@ -130,5 +183,5 @@
       <origin xyz="0 0 0" rpy="0 1.5707 1.5707"/>
       <geometry>
-        <cylinder radius="0.1" length="0.05"/>
+        <cylinder radius="0.5" length="0.5"/>
       </geometry>
     </collision>
@@ -136,53 +189,5 @@
       <origin xyz="0 0 0" rpy="0 1.5707 1.5707"/>
       <geometry>
-        <cylinder radius="0.1" length="0.05"/>
-      </geometry>
-    </visual>
-  </link>
-  <link name='chassis'>
-    <pose>0 0 0.1 0 0 0</pose>
-    <inertial>
-      <mass value="15.0"/>
-      <origin xyz="0.0 0 0" rpy=" 0 0 0"/>
-      <inertia
-          ixx="0.1" ixy="0" ixz="0"
-          iyy="0.1" iyz="0"
-          izz="0.1"
-      />
-    </inertial>
-    <collision name='collision'>
-      <origin xyz="0 0 0.05" rpy=" 0 0 0"/>
-      <geometry>
-        <cylinder length="0.2" radius="0.25"/>
-      </geometry>
-    </collision>
-    <visual name='chassis_visual'>
-      <origin xyz="0 0 0.05" rpy=" 0 0 0"/>
-      <geometry>
-       <cylinder length="0.2" radius="0.25"/>
-      </geometry>
-    </visual>
-    <collision name='back_caster_collision'>
-      <origin xyz="-0.15 0 -0.05" rpy=" 0 0 0"/>
-      <geometry>
-        <sphere radius="0.0499"/>
-      </geometry>
-    </collision>
-    <visual name='back_caster_visual'>
-      <origin xyz="-0.15 0 -0.05" rpy=" 0 0 0"/>
-      <geometry>
-        <sphere radius="0.05"/>
-      </geometry>
-    </visual>
-    <collision name='front_caster_collision'>
-      <origin xyz="0.15 0 -0.05" rpy=" 0 0 0"/>
-      <geometry>
-        <sphere radius="0.0499"/>
-      </geometry>
-    </collision>
-    <visual name='front_caster_visual'>
-      <origin xyz="0.15 0 -0.05" rpy=" 0 0 0"/>
-      <geometry>
-        <sphere radius="0.05"/>
+        <cylinder radius="0.5" length="0.5"/>
       </geometry>
     </visual>

Commit message: gripper

File: models/robot.xacro (robot description, xacro)
@@ -2,10 +2,15 @@
 <robot name="spw_robot" xmlns:xacro="http://www.ros.org/wiki/xacro">
   <xacro:include filename="$(find spw_robot)/models/robot.gazebo" />
-  <gazebo reference="base_center"><material>Gazebo/Blue</material></gazebo>
+  <gazebo reference="base_center"><material>Gazebo/Grey</material></gazebo>
   <gazebo reference="left_wheel"><material>Gazebo/Black</material></gazebo>
   <gazebo reference="right_wheel"><material>Gazebo/Black</material></gazebo>
-  <gazebo reference="link1"><material>Gazebo/Grey</material></gazebo>
-  <gazebo reference="link2"><material>Gazebo/Grey</material></gazebo>
-  <gazebo reference="link3"><material>Gazebo/Grey</material></gazebo>
+  <gazebo reference="left_wheel2"><material>Gazebo/Black</material></gazebo>
+  <gazebo reference="right_wheel2"><material>Gazebo/Black</material></gazebo>
+  <gazebo reference="link1"><material>Gazebo/Blue</material></gazebo>
+  <gazebo reference="link2"><material>Gazebo/Green</material></gazebo>
+  <gazebo reference="link3"><material>Gazebo/Yellow</material></gazebo>
+  <gazebo reference="link4"><material>Gazebo/White</material></gazebo>
+  <gazebo reference="link5"><material>Gazebo/Orange</material></gazebo>
+  <gazebo reference="link6"><material>Gazebo/Red</material></gazebo>
   <!-- FOOT PRINT -->
   <link name="robot_footprint"></link>
@@ -21,9 +26,5 @@
       <mass value="15.0"/>
       <origin xyz="0.0 0 0" rpy=" 0 0 0"/>
-      <inertia
-          ixx="0.1" ixy="0" ixz="0"
-          iyy="0.1" iyz="0"
-          izz="0.1"
-      />
+      <inertia ixx="0.1" ixy="0" ixz="0" iyy="0.1" iyz="0" izz="0.1" />
     </inertial>
     <collision name="collision">
@@ -40,41 +41,37 @@
     </visual>
   </link>
-  <!-- ARM TO ROTATE Z AXIS -->
-  <joint name="joint1" type="revolute">
+  <!-- ARM TO ROTATE AROUND Z AXIS -->
+  <joint name="joint1" type="continuous">
     <parent link="base_center"/>
     <child link="link1"/>
-    <origin xyz="0 0 1" rpy="0 0 0"/>
+    <origin xyz="0 0 0.1" rpy="0 0 0"/>
     <axis xyz="0 0 1"/>
-    <limit effort="100" velocity="100" lower="-1.5708" upper="1.5708"/>
   </joint>
   <link name="link1">
     <collision>
-      <origin xyz="0 0 0.05" rpy="0 0 0"/>
-      <geometry>
-        <cylinder length="1" radius="0.2"/>
-      </geometry>
-    </collision>
-    <visual>
-      <origin xyz="0 0 0.05" rpy="0 0 0"/>
-      <geometry>
-        <cylinder length="1" radius="0.2"/>
-      </geometry>
-    </visual>
-    <inertial>
-      <origin xyz="0 0 0.05" rpy="0 0 0"/>
+      <origin xyz="0 0 0.5" rpy="0 0 0"/>
+      <geometry>
+        <cylinder length="1" radius="0.1"/>
+      </geometry>
+    </collision>
+    <visual>
+      <origin xyz="0 0 0.5" rpy="0 0 0"/>
+      <geometry>
+        <cylinder length="1" radius="0.1"/>
+      </geometry>
+    </visual>
+    <inertial>
+      <origin xyz="0 0 0.5" rpy="0 0 0"/>
       <mass value="1"/>
-      <inertia
-        ixx="0.001" ixy="0.0" ixz="0.0"
-        iyy="0.001" iyz="0.0"
-        izz="0.001"/>
-    </inertial>
-  </link>
-  <!-- ARM TO ROTATE Y AXIS -->
+      <inertia ixx="0.1" ixy="0.0" ixz="0.0" iyy="0.1" iyz="0.0" izz="0.005"/>
+    </inertial>
+  </link>
+  <!-- ARM TO ROTATE ALONG Y AXIS -->
   <joint name="joint2" type="revolute">
     <parent link="link1"/>
     <child link="link2"/>
-    <origin xyz="0 0 0.1" rpy="0 0 0"/>
-    <axis xyz="0 1 0"/>
-    <limit effort="100" velocity="100" lower="-0.1" upper="1.5708"/>
+    <origin xyz="0 0 1" rpy="0 0 0"/>
+    <axis xyz="0 1 0"/>
+    <limit effort="1000" velocity="1000" lower="0" upper="1"/>
   </joint>
   <link name="link2">
@@ -94,8 +91,5 @@
       <origin xyz="0 0 0.5" rpy="0 0 0"/>
       <mass value="1"/>
-      <inertia
-        ixx="0.1" ixy="0.0" ixz="0.0"
-        iyy="0.1" iyz="0.0"
-        izz="0.005"/>
+      <inertia ixx="0.1" ixy="0.0" ixz="0.0" iyy="0.1" iyz="0.0" izz="0.005"/>
     </inertial>
   </link>
@@ -106,5 +100,5 @@
     <origin xyz="0 0 1" rpy="0 0 0"/>
     <axis xyz="0 1 0"/>
-    <limit effort="100" velocity="100" lower="-0.1" upper="3.1416"/>
+    <limit effort="1000" velocity="1000" lower="0" upper="1"/>
   </joint>
   <link name="link3">
@@ -123,48 +117,138 @@
     <inertial>
       <origin xyz="0 0 0.5" rpy="0 0 0"/>
-      <mass value="1"/>
-      <inertia
-        ixx="0.1" ixy="0.0" ixz="0.0"
-        iyy="0.1" iyz="0.0"
-        izz="0.005"/>
+      <mass value="0.6"/>
+      <inertia ixx="0.1" ixy="0.0" ixz="0.0" iyy="0.1" iyz="0.0" izz="0.005"/>
+    </inertial>
+  </link>
+  <!-- GRIPPER BASE -->
+  <joint name="joint4" type="revolute">
+    <parent link="link3"/>
+    <child link="link4"/>
+    <origin xyz="0 0 1" rpy="0 0 0"/>
+    <axis xyz="0 1 0"/>
+    <limit effort="10" velocity="10" lower="-1.5708" upper="1.5708"/>
+  </joint>
+  <link name="link4">
+    <collision>
+      <origin xyz="0 0 0" rpy="1.5708 0 0"/>
+      <geometry>
+        <cylinder length="0.4" radius="0.04"/>
+      </geometry>
+    </collision>
+    <visual>
+      <origin xyz="0 0 0" rpy="1.5708 0 0"/>
+      <geometry>
+        <cylinder length="0.4" radius="0.04"/>
+      </geometry>
+    </visual>
+    <inertial>
+      <origin xyz="0 0 0" rpy="1.5708 0 0"/>
+      <mass value="0.4"/>
+      <inertia ixx="0.05" ixy="0.0" ixz="0.0" iyy="0.002" iyz="0.0" izz="0.05"/>
+    </inertial>
+  </link>
+  <!-- GRIPPER LEFT-->
+  <joint name="joint5" type="prismatic">
+    <parent link="link4"/>
+    <child link="link5"/>
+    <origin xyz="0 0.16 0" rpy="0 0 0"/>
+    <axis xyz="0 1 0"/>
+    <limit effort="1000" velocity="1000" lower="-0.1" upper="0.0"/>
+  </joint>
+  <link name="link5">
+    <collision>
+      <origin xyz="0 0 0.15" rpy="0 0 0"/>
+      <geometry>
+        <cylinder length="0.3" radius="0.04"/>
+      </geometry>
+    </collision>
+    <visual>
+      <origin xyz="0 0 0.15" rpy="0 0 0"/>
+      <geometry>
+        <cylinder length="0.3" radius="0.04"/>
+      </geometry>
+    </visual>
+    <inertial>
+      <origin xyz="0 0 0.15" rpy="0 0 0"/>
+      <mass value="0.2"/>
+      <inertia ixx="0.02" ixy="0.0" ixz="0.0" iyy="0.02" iyz="0.0" izz="0.001"/>
+    </inertial>
+  </link>
+  <!-- GRIPPER RIGHT -->
+  <joint name="joint6" type="prismatic">
+    <parent link="link4"/>
+    <child link="link6"/>
+    <origin xyz="0 -0.16 0" rpy="0 0 0"/>
+    <axis xyz="0 1 0"/>
+    <limit effort="1000" velocity="1000" lower="0.0" upper="0.1"/>
+  </joint>
+  <link name="link6">
+    <collision>
+      <origin xyz="0 0 0.15" rpy="0 0 0"/>
+      <geometry>
+        <cylinder length="0.3" radius="0.04"/>
+      </geometry>
+    </collision>
+    <visual>
+      <origin xyz="0 0 0.15" rpy="0 0 0"/>
+      <geometry>
+        <cylinder length="0.3" radius="0.04"/>
+      </geometry>
+    </visual>
+    <inertial>
+      <origin xyz="0 0 0.15" rpy="0 0 0"/>
+      <mass value="0.2"/>
+      <inertia ixx="0.02" ixy="0.0" ixz="0.0" iyy="0.02" iyz="0.0" izz="0.001"/>
     </inertial>
   </link>
   <!-- WHEELS -->
-  <joint name="left_wheel_hinge" type="continuous">
-    <origin xyz="0 0.5 0" rpy="0 0 0" />
+  <joint name="left_wheel_hinge" type="fixed">
+    <origin xyz="0.35 0.5 -0.3" rpy="0 0 0" />
     <parent link="base_center"/>
     <child link="left_wheel" />
     <axis xyz="0 1 0" rpy="0 0 0" />
-    <limit effort="10000" velocity="1000" />
+    <limit effort="1000" velocity="1000" />
     <dynamics damping="1.0" friction="1.0" />
   </joint>
-  <joint name="right_wheel_hinge" type="continuous">
-    <origin xyz="0 -0.5 0" rpy="0 0 0" />
+  <joint name="right_wheel_hinge" type="fixed">
+    <origin xyz="0.35 -0.5 -0.3" rpy="0 0 0" />
     <parent link="base_center"/>
     <child link="right_wheel" />
     <axis xyz="0 1 0" rpy="0 0 0" />
-    <limit effort="10000" velocity="1000" />
+    <limit effort="1000" velocity="1000" />
     <dynamics damping="1.0" friction="1.0" />
   </joint>
+  <joint name="left_wheel_hinge2" type="fixed">
+    <origin xyz="-0.35 0.5 -0.3" rpy="0 0 0" />
+    <parent link="base_center"/>
+    <child link="left_wheel2" />
+    <axis xyz="0 1 0" rpy="0 0 0" />
+    <limit effort="1000" velocity="1000" />
+    <dynamics damping="1.0" friction="1.0" />
+  </joint>
+  <joint name="right_wheel_hinge2" type="fixed">
+    <origin xyz="-0.35 -0.5 -0.3" rpy="0 0 0" />
+    <parent link="base_center"/>
+    <child link="right_wheel2" />
+    <axis xyz="0 1 0" rpy="0 0 0" />
+    <limit effort="1000" velocity="1000" />
+    <dynamics damping="1.0" friction="1.0" />
+  </joint>
   <link name="left_wheel">
     <inertial>
       <mass value="5"/>
       <origin xyz="0 0 0" rpy="0 1.5707 1.5707"/>
-      <inertia
-        ixx="0.1" ixy="0.0" ixz="0.0"
-        iyy="0.1" iyz="0.0"
-        izz="0.1"
-      />
-    </inertial>
-    <collision>
-      <origin xyz="0 0 0" rpy="0 1.5707 1.5707"/>
-      <geometry>
-        <cylinder radius="0.5" length="0.5"/>
-      </geometry>
-    </collision>
-    <visual>
-      <origin xyz="0 0 0" rpy="0 1.5707 1.5707"/>
-      <geometry>
-        <cylinder radius="0.5" length="0.5"/>
+      <inertia ixx="0.1" ixy="0.0" ixz="0.0" iyy="0.1" iyz="0.0" izz="0.1" />
+    </inertial>
+    <collision>
+      <origin xyz="0 0 0" rpy="0 1.5707 1.5707"/>
+      <geometry>
+        <cylinder radius="0.3" length="0.5"/>
+      </geometry>
+    </collision>
+    <visual>
+      <origin xyz="0 0 0" rpy="0 1.5707 1.5707"/>
+      <geometry>
+        <cylinder radius="0.3" length="0.5"/>
       </geometry>
     </visual>
@@ -174,20 +258,54 @@
       <mass value="5"/>
       <origin xyz="0 0 0" rpy="0 1.5707 1.5707"/>
-      <inertia
-        ixx="0.1" ixy="0.0" ixz="0.0"
-        iyy="0.1" iyz="0.0"
-        izz="0.1"
-      />
-    </inertial>
-    <collision>
-      <origin xyz="0 0 0" rpy="0 1.5707 1.5707"/>
-      <geometry>
-        <cylinder radius="0.5" length="0.5"/>
-      </geometry>
-    </collision>
-    <visual>
-      <origin xyz="0 0 0" rpy="0 1.5707 1.5707"/>
-      <geometry>
-        <cylinder radius="0.5" length="0.5"/>
+      <inertia ixx="0.1" ixy="0.0" ixz="0.0" iyy="0.1" iyz="0.0" izz="0.1" />
+    </inertial>
+    <collision>
+      <origin xyz="0 0 0" rpy="0 1.5707 1.5707"/>
+      <geometry>
+        <cylinder radius="0.3" length="0.5"/>
+      </geometry>
+    </collision>
+    <visual>
+      <origin xyz="0 0 0" rpy="0 1.5707 1.5707"/>
+      <geometry>
+        <cylinder radius="0.3" length="0.5"/>
+      </geometry>
+    </visual>
+  </link>
+  <link name="left_wheel2">
+    <inertial>
+      <mass value="5"/>
+      <origin xyz="0 0 0" rpy="0 1.5707 1.5707"/>
+      <inertia ixx="0.1" ixy="0.0" ixz="0.0" iyy="0.1" iyz="0.0" izz="0.1" />
+    </inertial>
+    <collision>
+      <origin xyz="0 0 0" rpy="0 1.5707 1.5707"/>
+      <geometry>
+        <cylinder radius="0.3" length="0.5"/>
+      </geometry>
+    </collision>
+    <visual>
+      <origin xyz="0 0 0" rpy="0 1.5707 1.5707"/>
+      <geometry>
+        <cylinder radius="0.3" length="0.5"/>
+      </geometry>
+    </visual>
+  </link>
+  <link name="right_wheel2">
+    <inertial>
+      <mass value="5"/>
+      <origin xyz="0 0 0" rpy="0 1.5707 1.5707"/>
+      <inertia ixx="0.1" ixy="0.0" ixz="0.0" iyy="0.1" iyz="0.0" izz="0.1" />
+    </inertial>
+    <collision>
+      <origin xyz="0 0 0" rpy="0 1.5707 1.5707"/>
+      <geometry>
+        <cylinder radius="0.3" length="0.5"/>
+      </geometry>
+    </collision>
+    <visual>
+      <origin xyz="0 0 0" rpy="0 1.5707 1.5707"/>
+      <geometry>
+        <cylinder radius="0.3" length="0.5"/>
       </geometry>
     </visual>
